File: hardware/ARCS-PD-M-0C072R020M064/8Bit_Shifted_Input.sch (KiCad schematic (older format))
At the start: 173 parts, among them J501 Input_Terminal_01x02, J502 Input_Terminal_01x02, J503 Input_Terminal_01x02, J504 Input_Terminal_01x02, J505 Input_Terminal_01x02, J506 Input_Terminal_01x02, J507 Input_Terminal_01x02, J508 Input_Terminal_01x02, Q501 PMBT3906, Q502 PMBT3906, Q503 PMBT3906, Q504 PMBT3906, Q505 PMBT3906, Q506 PMBT3906, Q507 PMBT3906, Q508 PMBT3906, Q509 PMBT3906, Q510 PMBT3906, Q511 PMBT3906, Q512 PMBT3906, Q513 PMBT3906, Q514 PMBT3906, Q515 PMBT3906, Q516 PMBT3906, Q517 PMBT3906, Q518 PMBT3906, Q519 PMBT3906, Q520 PMBT3906, Q521 PMBT3906, Q522 PMBT3906, Q523 PMBT3906, Q524 PMBT3906, Q525 PMBT3906, Q526 PMBT3906, Q527 PMBT3906, Q528 PMBT3906, Q529 PMBT3906, Q530 PMBT3906, Q531 PMBT3906, Q532 PMBT3906, SW501 SW_DIP_x02, SW502 SW_DIP_x02, SW503 SW_DIP_x02, SW504 SW_DIP_x02, SW505 SW_DIP_x02, SW506 SW_DIP_x02, SW507 SW_DIP_x02, SW508 SW_DIP_x02, U501 74HC00, U502 LM324, U503 LM324, U504 74HC74, U505 74HC74, U506 LM324, U507 74LVC1G125, U508 LM324, U509 74HC4051, U510 74HC4051, U511 74HC4051, U512 74HC4051, U513 74HC4051, U514 74HC4051, U515 74HC4051, U516 74HC4051, U517 74HC4051

Commit message: Make changes to STM32F103C8 and add STM32F103VE based PD system.
Parts:
- added R? (x16): 10k, symbol Device:R
- U507: symbol 74xGxx-custom:74LVC1G125-Custom -> ARCS-PD-M-0C072R020M064-rescue:74LVC1G125-Custom-74xGxx-custom
Connections:
- net labels added: A00, A01, A02, A10, A11, A12, A20, A21, A22, A30, A31, A32, A40, A41, A42, A50, A51, A52, A60, A61, A62, A70, A71, A72
- wire segments 825 -> 806
Other:
- note added: "1ST STAGE 8 CHANNEL SIGNAL BUFFER"
- note added: "2ND STAGE 8 CHANNEL SIGNAL BUFFER"
- note added: "4 BIT COUNTER"
- note added: "CHENNEL SELECT MUX"
- note added: "COUNTER OVERFLOW DETECTION"
- note added: "INPUT CONNECTORS"
- note removed: "A7 | A0\nA6 | A1\nA5 | A2\nA4 | A3"
- moved on the sheet: C501, C502, C503, J501, J502, J503, J504, J505, J506, J507, J508, R501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
