File: hardware/ARCS-PD-M-0C072R020M064/8Bit_Shifted_Output.sch (KiCad schematic (older format))
At the start: 75 parts, among them J201 Conn_01x02, J202 Conn_01x02, J203 Conn_01x02, J204 Conn_01x02, J205 Conn_01x02, J206 Conn_01x02, J207 Conn_01x02, J208 Conn_01x02, K201 G6S-2, K202 G6S-2, K203 G6S-2, K204 G6S-2, K205 G6S-2, K206 G6S-2, K207 G6S-2, K208 G6S-2, Q201 2N7002, Q202 2N7002, Q203 2N7002, Q204 2N7002, Q205 2N7002, Q206 2N7002, Q207 2N7002, Q208 2N7002, U201 74HC74, U202 74HC374, U203 74HC00, U204 74HC74, U205 74HC374, U206 74LVC1G125, U207 74HC4051, U208 74LVC1G125, U209 74LVC1G125, U210 74LVC1G125, U211 74LVC1G125, U212 74LVC1G125, U213 74LVC1G125, U214 74LVC1G125, U215 74LVC1G125

Commit message: Make changes to STM32F103C8 and add STM32F103VE based PD system.
Parts:
- U206, U208, U209, U210, U211, U212, U213, U214, U215: symbol 74xGxx-custom:74LVC1G125-Custom -> ARCS-PD-M-0C072R020M064-rescue:74LVC1G125-Custom-74xGxx-custom
Changed lines of the file:
@@
 Connection ~ 7150 5150
 $Comp
-L 74xGxx-custom:74LVC1G125-Custom U?
+L ARCS-PD-M-0C072R020M064-rescue:74LVC1G125-Custom-74xGxx-custom U?
 U 1 1 5E07AD80
 P 6400 5750
@@
 Connection ~ 4250 4050
 $Comp
-L 74xGxx-custom:74LVC1G125-Custom U?
+L ARCS-PD-M-0C072R020M064-rescue:74LVC1G125-Custom-74xGxx-custom U?
 U 1 1 5E07AE34
 P 4900 4500
@@
 Connection ~ 9650 5150
 $Comp
-L 74xGxx-custom:74LVC1G125-Custom U?
+L ARCS-PD-M-0C072R020M064-rescue:74LVC1G125-Custom-74xGxx-custom U?
 U 1 1 5E07AF08
 P 8900 5750
@@
 Connection ~ 12100 5150
 $Comp
-L 74xGxx-custom:74LVC1G125-Custom U?
+L ARCS-PD-M-0C072R020M064-rescue:74LVC1G125-Custom-74xGxx-custom U?
 U 1 1 5E07AF52
 P 11350 5750
@@
 Connection ~ 14600 5150
 $Comp
-L 74xGxx-custom:74LVC1G125-Custom U?
+L ARCS-PD-M-0C072R020M064-rescue:74LVC1G125-Custom-74xGxx-custom U?
 U 1 1 5E07AF9C
 P 13850 5750
@@
 Connection ~ 7500 7450
 $Comp
-L 74xGxx-custom:74LVC1G125-Custom U?
+L ARCS-PD-M-0C072R020M064-rescue:74LVC1G125-Custom-74xGxx-custom U?
 U 1 1 5E07AFE6
 P 6450 8050
@@
 Connection ~ 9950 7450
 $Comp
-L 74xGxx-custom:74LVC1G125-Custom U?
+L ARCS-PD-M-0C072R020M064-rescue:74LVC1G125-Custom-74xGxx-custom U?
 U 1 1 5E07B030
 P 8900 8050
@@
 Connection ~ 12400 7450
 $Comp
-L 74xGxx-custom:74LVC1G125-Custom U?
+L ARCS-PD-M-0C072R020M064-rescue:74LVC1G125-Custom-74xGxx-custom U?
 U 1 1 5E07B07A
 P 11350 8050
@@
 Connection ~ 14900 7450
 $Comp
-L 74xGxx-custom:74LVC1G125-Custom U?
+L ARCS-PD-M-0C072R020M064-rescue:74LVC1G125-Custom-74xGxx-custom U?
 U 1 1 5E07B0C4
 P 13850 8050
