File: hardware/ARCS-PD-M-0C072R020M064/ARCS-PD-M-0C072R020M064.sch (KiCad schematic (older format))
At the start: 24 parts, among them J101 USB_B, J102 Conn_01x02, J103 Conn_01x02, J104 Conn_01x02_PWR, J105 Conn_01x02_PWR, J106 JST-XH-01X02, J107 Conn_01x02, U101 AMS1117-3.3, U102 74LVC1G125

Commit message: Make changes to STM32F103C8 and add STM32F103VE based PD system.
Parts:
- U102: symbol 74xGxx-custom:74LVC1G125-Custom -> ARCS-PD-M-0C072R020M064-rescue:74LVC1G125-Custom-74xGxx-custom
Connections:
- wire segments 85 -> 83
Changed lines of the file:
@@
 $EndComp
 $Comp
-L 74xGxx-custom:74LVC1G125-Custom U102
+L ARCS-PD-M-0C072R020M064-rescue:74LVC1G125-Custom-74xGxx-custom U102
 U 1 1 67FE5EA1
 P 5300 4650
@@
 Wire Wire Line
 	4600 4250 4750 4250
-Wire Wire Line
-	4750 4250 4750 4550
-Wire Wire Line
-	4650 4550 4650 4500
 $Comp
 L power:+3.3V #PWR0104
 U 1 1 68136D17
-P 4450 4200
-F 0 "#PWR0104" H 4450 4050 50  0001 C CNN
-F 1 "+3.3V" V 4465 4328 50  0000 L CNN
-F 2 "" H 4450 4200 50  0001 C CNN
-F 3 "" H 4450 4200 50  0001 C CNN
-	1    4450 4200
+P 4500 4200
+F 0 "#PWR0104" H 4500 4050 50  0001 C CNN
+F 1 "+3.3V" V 4515 4328 50  0000 L CNN
+F 2 "" H 4500 4200 50  0001 C CNN
+F 3 "" H 4500 4200 50  0001 C CNN
+	1    4500 4200
 	0    -1   -1   0
 $EndComp
 Wire Wire Line
-	4450 4200 4650 4200
-Wire Wire Line
-	4650 4200 4650 4400
-Wire Wire Line
 	4300 4450 4100 4450
-Wire Wire Line
-	4650 4550 4750 4550
-Connection ~ 4650 4550
 $Comp
 L Device:R R102
@@
 Wire Wire Line
 	4200 4650 4200 4750
-Wire Wire Line
-	3500 5100 4650 5100
-Wire Wire Line
-	4650 4550 4650 5100
 Connection ~ 3500 5100
 Wire Wire Line
@@
 $EndSheet
 $Sheet
-S 7400 3000 1700 1400
+S 600  1850 1700 1400
 U 5E6E13CF
 F0 "Sheet5E6E13CE" 50
@@
 Wire Wire Line
 	4300 2650 5200 2650
+Wire Wire Line
+	4500 4200 4500 4300
+Wire Wire Line
+	4500 4600 4750 4600
+Wire Wire Line
+	4750 4250 4750 4600
+Wire Wire Line
+	4750 5100 4750 4600
+Wire Wire Line
+	3500 5100 4750 5100
+Connection ~ 4750 4600
 $EndSCHEMATC
