File: hardware/ARCS-PD-M-0C072R020M064/TWCL_Comm_Interface.sch (KiCad schematic (older format))
At the start: 30 parts, among them J401 XLR3_Ground, J402 XLR3_Ground, J403 XLR3_Ground, Q401 2N7002, Q402 2N7002, Q403 2N7002, Q404 2N7002, U401 74LVC1G125, U402 74LVC1G125, U403 74LVC1G00, U404 74LVC1G125, U405 74LVC1G125, U406 74LVC1G125, U407 74LVC1G00, U408 74LVC1G00

Commit message: Make changes to STM32F103C8 and add STM32F103VE based PD system.
Parts:
- U401, U402, U404, U405, U406: symbol 74xGxx-custom:74LVC1G125-Custom -> ARCS-PD-M-0C072R020M064-rescue:74LVC1G125-Custom-74xGxx-custom
- U403, U407, U408: symbol 74xGxx-custom:74LVC1G00 -> ARCS-PD-M-0C072R020M064-rescue:74LVC1G00-74xGxx-custom
Changed lines of the file:
@@
 $EndComp
 $Comp
-L 74xGxx-custom:74LVC1G00 U?
+L ARCS-PD-M-0C072R020M064-rescue:74LVC1G00-74xGxx-custom U?
 U 1 1 5E529A58
 P 6650 4500
@@
 T3-TX
 $Comp
-L 74xGxx-custom:74LVC1G125-Custom U?
+L ARCS-PD-M-0C072R020M064-rescue:74LVC1G125-Custom-74xGxx-custom U?
 U 1 1 5E529A84
 P 6000 4950
@@
 $EndComp
 $Comp
-L 74xGxx-custom:74LVC1G00 U?
+L ARCS-PD-M-0C072R020M064-rescue:74LVC1G00-74xGxx-custom U?
 U 1 1 5E529ADC
 P 3950 2000
@@
 T2-TX
 $Comp
-L 74xGxx-custom:74LVC1G125-Custom U?
+L ARCS-PD-M-0C072R020M064-rescue:74LVC1G125-Custom-74xGxx-custom U?
 U 1 1 5E529AF1
 P 3300 2450
@@
 $EndComp
 $Comp
-L 74xGxx-custom:74LVC1G125-Custom U?
+L ARCS-PD-M-0C072R020M064-rescue:74LVC1G125-Custom-74xGxx-custom U?
 U 1 1 5E529B0C
 P 4750 3900
@@
 $EndComp
 $Comp
-L 74xGxx-custom:74LVC1G125-Custom U?
+L ARCS-PD-M-0C072R020M064-rescue:74LVC1G125-Custom-74xGxx-custom U?
 U 1 1 5E529B13
 P 3300 3450
@@
 $EndComp
 $Comp
-L 74xGxx-custom:74LVC1G00 U?
+L ARCS-PD-M-0C072R020M064-rescue:74LVC1G00-74xGxx-custom U?
 U 1 1 5E529B44
 P 6650 2400
@@
 T1-TX
 $Comp
-L 74xGxx-custom:74LVC1G125-Custom U?
+L ARCS-PD-M-0C072R020M064-rescue:74LVC1G125-Custom-74xGxx-custom U?
 U 1 1 5E529B70
 P 6000 2850
