File: hardware/ARCS-CARDS/I-16-4/AII4.sch (KiCad schematic (older format))
At the start: 63 parts

Commit message: Create analog input interface card.
Parts:
- removed FB?: Ferrite_Bead, symbol Device:Ferrite_Bead
- removed Q?: BSS83P, Package_TO_SOT_SMD:SOT-23, symbol Transistor_FET:BSS83P
- removed Q?: 2N7002, Package_TO_SOT_SMD:SOT-23, symbol Transistor_FET:2N7002
- removed R? (x2): 10k, symbol Device:R
- added C? (x2): 10n, symbol Device:C
- added C? (x5): 100n, symbol Device:C
- added D? (x4): 1SMA5918BT3G, symbol Device:D_Zener_ALT
- added FB?: Ferrite_Bead, symbol Device:Ferrite_Bead
- added J? (x4): Conn_01x01, symbol Connector_Generic:Conn_01x01
- added R? (x4): 10k, symbol Device:R
- added RV?: 500R, symbol Device:R_POT_TRIM
- added U?: NE555, symbol Timer:NE555
- added U?: 74LVC1G32, symbol 74xGxx_custom:74LVC1G32
- added U? (x3): 74LVC1G125, symbol 74xGxx_custom:74LVC1G125
- added U? (x2): 74HC573, symbol 74xx:74LS573
- added U?: 74LVC1G00, symbol 74xGxx_custom:74LVC1G00
Connections:
- net +5V: now also C?.1, C?.1, C?.1, C?.1, C?.1, RV?.1, U?.2, U?.20 (VCC), U?.20 (VCC), U?.4 (R), U?.5 (PWR), U?.5 (PWR), U?.5 (PWR), U?.8 (VCC)
- net C1-12V-SEL: now also Q?.1 (G), R?.1
- net C1-24V-SEL: now also Q?.1 (G), R?.2
- net C2-12V-SEL: now also Q?.1 (G), R?.1
- net C3-12V-SEL: now also Q?.1 (G), R?.1
- net C4-12V-SEL: now also Q?.1 (G), R?.1
- net Earth: now also C?.2, C?.2, C?.2, C?.2, C?.2, C?.2, C?.2, FB?.1, J?.1 (Pin_1), J?.1 (Pin_1), J?.1 (Pin_1), U?.1 (GND), U?.1 (OE), U?.1 (OE), U?.10 (GND), U?.10 (GND), U?.3 (GND), U?.3 (GND), U?.3 (GND), U?.5 (D3), U?.5 (D3), U?.6 (D4), U?.6 (D4), U?.7 (D5), U?.7 (D5), U?.8 (D6), U?.8 (D6), U?.9 (D7), U?.9 (D7); no longer Q?.2 (S), Q?.2 (S), Q?.2 (S), Q?.2 (S), Q?.2 (S), Q?.2 (S), Q?.2 (S), Q?.2 (S)
- net GNDA: now also Q?.2 (S), Q?.2 (S), Q?.2 (S), Q?.2 (S), Q?.2 (S), Q?.2 (S), Q?.2 (S), Q?.2 (S), D?.2 (A), D?.2 (A), D?.2 (A), D?.2 (A), R?.2, R?.2, R?.2, R?.2
- net IN1: now also R?.1; no longer U?.12 (+), U?.4 (+), U?.9 (+)
- net IN-RNG-CARRY-OUT: now reaches U?.12 (Q7), U?.9 (D7)
- net at R?.1, R?.1, R?.2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: now also D?.1 (K) (x4)
- net EOC: now reaches U?.10 (EOC)
- net EOC: now also U?.1
- net at R?.1, U?.15 (PE), U?.15 (PE): now also U?.1, U?.4
- net at R?.1, U?.7 (Clk), U?.7 (Clk): now also U?.4
- net IN-SEL-A0: now reaches U?.1 (A0)
- net IN-SEL-A0: now also U?.19 (Q0)
- net IN-SEL-A2: now reaches U?.15 (A2)
- net IN-SEL-A2: now also U?.17 (Q2)
- net IN-SEL-A1: now reaches U?.16 (A1)
- net IN-SEL-A1: now also U?.18 (Q1)
- net C2-24V-SEL: now reaches Q?.1 (G), R?.2
- net C3-24V-SEL: now reaches Q?.1 (G), R?.2
- net C4-24V-SEL: now reaches Q?.1 (G), R?.2
- net CARRY-IN renamed OUT-CARRY-IN
- net CARRY-OUT renamed OUT-CARRY-OUT
- net SEL-RNG-BIT renamed IN-RNG-CARRY-IN
- net SET-RNG-PUSH renamed IN-RNG-PUSH
- net SET-RNG-SHIFT renamed IN-RNG-SHIFT
- new net: C?.1, RV?.3, U?.2 (TR), U?.6 (THR)
- new net: C?.1, U?.5 (CV)
- new net: RV?.2, U?.7 (DIS)
- new net: U?.2, U?.4
- new net: U?.1, U?.1, U?.2, U?.4
- new net: U?.18 (Q1), U?.3 (D1), U?.4 (D2)
- new net: U?.19 (Q0), U?.2 (D0), U?.3 (D1)
- new net: FB?.2, J?.1 (Pin_1)
- new net: U?.3 (GND), U?.3 (GND)
- new net: U?.5 (PWR), U?.5 (PWR)
- new net AQ-CLK: U?.3 (Q), U?.~ (RESET)
- new net IN-SEL-CARRY-IN: U?.2 (D0)
- new net IN-SEL-CARRY-OUT: U?.17 (Q2), U?.4 (D2)
- new net IN-SEL-PUSH: U?.11 (Load)
- new net IN-SEL-SHIFT: U?.11 (Load)
- new net IN2: R?.1, U?.4 (+)
- new net IN3: R?.1, U?.9 (+)
- new net IN4: R?.1, U?.12 (+)
- no-connect marks 7 -> 14
Other:
- note added: "0 | 0 > 0-24V\n0 | 1 > 0-5V\n1 | 0 > FORBIDDEN\n1 | 1 > 0-12V"
- note added: "0 | 0 | 0 > IN1\n1 | 0 | 0 > IN2\n0 | 1 | 0 > IN3\n1 | 1 | 0 > IN4\n0 | 0 | 1 > NC\n1 | 0 | 1 > NC\n0 | 1 | 1 > NC\n1 | 1 | 1 > NC"
- note added: "ACQUISITION CLOCK"
- note added: "CAUTION !!! Make sure that correct\nrange is selected for the input. If lower\nrange is selected for a high input (for\nexample 0-5V and input is at 24V) it\nis posible to demage MUX or ADC."
- note added: "Every input has 2 bits reserved for \nrange selection. For IN1, BIT0 and \nBIT1 are used, for IN2, BIT2 and BIT3 \nare used and so on."
- note added: "Generate a 100kHz square wave clock signal\nfor the ADC. Conversion is done every 3th\nclock pulse and is automatically parsed to\nthe output buffer. If OUT-RW is set to read,\nresult of ADC will not be added to the output\nbuffer."
- note added: "IN-ENG-CARRY-OUT - Carry the last bit \nof the buffer register to the next\nregister in the chain."
- note added: "IN-RNG-CARRY-IN - Set a bit that will be \nshifted into buffer register. This pin can be\nconnected to a MCU or it can be connected\nto a CARRY-OUT of the previous chain."
- note added: "IN-RNG-PUSH - Push bits from the \nbuffer register to the state \nregister. With this action, input range\nwill be set."
- note added: "IN-RNG-SHIFT - Shift a buffer register\none place to the right."
- note added: "IN-SEL-CARRY-IN - Set a bit that will be \nshifted into buffer register. This pin can be\nconnected to a MCU or it can be connected\nto a CARRY-OUT of the previous chain."
- note added: "IN-SEL-CARRY-OUT - Carry the last bit \nof the buffer register to the next\nregister in the chain."
- note added: "IN-SEL-PUSH - Push bits from the \nbuffer register to the state \nregister. With this action, input range\nwill be set."
- note added: "IN-SEL-SHIFT - Shift a buffer register\none place to the right."
- note added: "INPUT RANGE SELECT REGISTER"
- note added: "INPUT SELECT REGISTER"
- note added: "OUT-CARRY-IN - Set a bit that will be \nshifted into buffer register. This pin can be\nconnected to a MCU or it can be connected\nto a CARRY-OUT of the previous chain."
- note added: "OUT-CARRY-OUT - Carry the last bit \nof the buffer register to the next\nregister in the chain or input of the MCU."
- note added: "OUT-RW - Set output register to read/write \nstate. If in write state, on next clock pulse\n(on OUT-SHIFT pin) output of the ADC will be\nadded to the output buffer register. If in\nread state, on next clock pulse output buffer\nregister will be shifted one place to the right."
- note added: "OUT-SHIFT - Shift a buffer register\none place to the right."
- note added: "OUTPUT REGISTER"
- note added: "This register is used to parse an ADC resault\nto the MCU as a sequence of bits. Sequence\nis parsed with LSB first. With each I-16-4 card\ncalibration paper will be provided with transfer\nfunction for each range. In this way, 16-bit\nbinary number can be converted into the voltage\nmeasured by ADC."
- note added: "This regitesr determens which input\nwill be parsed to the ADC. Only 1 can\nbe connected at a time."
- moved on the sheet: C?, Q?, R?, U?, U?A, U?B, U?C, U?D, U?E

Commit message: Create analog input interface card.
Parts:
- U?: symbol ADC:MAX1165 -> ARCS-CARDS-I-16-4-rescue:MAX1165-ADC
- U?: symbol MUX-DMUX:ADG708 -> ARCS-CARDS-I-16-4-rescue:ADG708-MUX-DMUX
- U?: symbol 74xGxx_custom:74LVC1G32 -> ARCS-CARDS-I-16-4-rescue:74LVC1G32-74xGxx_custom
- U? (x3): symbol 74xGxx_custom:74LVC1G125 -> ARCS-CARDS-I-16-4-rescue:74LVC1G125-74xGxx_custom
- U? (x4): symbol OPAmps:LM324QT -> ARCS-CARDS-I-16-4-rescue:LM324QT-OPAmps
- U?: symbol 74xGxx_custom:74LVC1G00 -> ARCS-CARDS-I-16-4-rescue:74LVC1G00-74xGxx_custom
Changed lines of the file:
@@
 $EndDescr
 $Comp
-L OPAmps:LM324QT U?
+L ARCS-CARDS-I-16-4-rescue:LM324QT-OPAmps U?
 U 1 1 5CF711FD
 P 1950 1150
@@
 $EndComp
 $Comp
-L OPAmps:LM324QT U?
+L ARCS-CARDS-I-16-4-rescue:LM324QT-OPAmps U?
 U 2 1 5CF7122F
 P 1950 2000
@@
 $EndComp
 $Comp
-L OPAmps:LM324QT U?
+L ARCS-CARDS-I-16-4-rescue:LM324QT-OPAmps U?
 U 3 1 5CF7129E
 P 1950 2850
@@
 $EndComp
 $Comp
-L OPAmps:LM324QT U?
+L ARCS-CARDS-I-16-4-rescue:LM324QT-OPAmps U?
 U 4 1 5CF71324
 P 1950 3700
@@
 $EndComp
 $Comp
-L MUX-DMUX:ADG708 U?
+L ARCS-CARDS-I-16-4-rescue:ADG708-MUX-DMUX U?
 U 1 1 5CAFA832
 P 4550 1800
@@
 	6100 8550 6100 10800
 $Comp
-L ADC:MAX1165 U?
+L ARCS-CARDS-I-16-4-rescue:MAX1165-ADC U?
 U 1 1 5CA5F3FB
 P 5700 2000
@@
 	12100 8500 11400 8500
 $Comp
-L 74xGxx_custom:74LVC1G32 U?
+L ARCS-CARDS-I-16-4-rescue:74LVC1G32-74xGxx_custom U?
 U 1 1 5CD12A81
 P 11450 4350
@@
 $EndComp
 $Comp
-L 74xGxx_custom:74LVC1G125 U?
+L ARCS-CARDS-I-16-4-rescue:74LVC1G125-74xGxx_custom U?
 U 1 1 5CD1927B
 P 12350 4400
@@
 	4900 2100 5200 2100
 $Comp
-L 74xGxx_custom:74LVC1G00 U?
+L ARCS-CARDS-I-16-4-rescue:74LVC1G00-74xGxx_custom U?
 U 1 1 5DF5C728
 P 13200 4400
+AR Path="/5DF5C728" Ref="U?"  Part="1"
+AR Path="/5CF1139E/5DF5C728" Ref="U?"  Part="1"
 F 0 "U?" H 13200 4800 50  0000 C CNN
 F 1 "74LVC1G00" H 13200 4700 50  0000 C CNN
@@
 	13700 4350 13500 4350
 $Comp
-L 74xGxx_custom:74LVC1G125 U?
+L ARCS-CARDS-I-16-4-rescue:74LVC1G125-74xGxx_custom U?
 U 1 1 5E02F9C1
 P 12750 3900
@@
 $EndComp
 $Comp
-L 74xGxx_custom:74LVC1G125 U?
+L ARCS-CARDS-I-16-4-rescue:74LVC1G125-74xGxx_custom U?
 U 1 1 5E0304DB
 P 12750 3450
